Commit message: add ee and scene camera

File: franka_ros/franka_description/robots/panda/panda.urdf.xacro (robot description, xacro)
@@ -6,3 +6,87 @@
                       joint_limits="${xacro.load_yaml('$(find franka_description)/robots/panda/joint_limits.yaml')}">
   </xacro:franka_robot>
+  <link name="ee_camera_link">
+    <inertial>
+      <mass value="0.1"/>
+      <origin xyz="0 0 0"/>
+      <inertia ixx="1e-5" ixy="0" ixz="0" iyy="1e-5" iyz="0" izz="1e-5"/>
+    </inertial>
+    <visual>
+      <geometry>
+        <box size="0.02 0.02 0.02"/>
+      </geometry>
+    </visual>
+  </link>
+  <joint name="ee_camera_joint" type="fixed">
+    <parent link="panda_hand"/>
+    <child link="ee_camera_link"/>
+    <origin xyz="0.04 0 0.05" rpy="0 -2.1 0"/>
+  </joint>
+  <gazebo reference="ee_camera_link">
+  <sensor type="camera" name="ee_camera">
+    <update_rate>30.0</update_rate>
+    <camera>
+      <horizontal_fov>1.3962634</horizontal_fov>
+      <image>
+        <width>640</width>
+        <height>480</height>
+        <format>R8G8B8</format>
+      </image>
+      <clip>
+        <near>0.01</near>
+        <far>100</far>
+      </clip>
+    </camera>
+    <plugin name="camera_controller" filename="libgazebo_ros_camera.so">
+      <alwaysOn>true</alwaysOn>
+      <updateRate>30.0</updateRate>
+      <cameraName>ee_camera</cameraName>
+      <imageTopicName>image_raw</imageTopicName>
+      <cameraInfoTopicName>camera_info</cameraInfoTopicName>
+      <frameName>ee_camera_link</frameName>
+    </plugin>
+  </sensor>
+  </gazebo>
+  <link name="scene_camera_link">
+    <inertial>
+      <mass value="0.1"/>
+      <origin xyz="0 0 0"/>
+      <inertia ixx="1e-5" ixy="0" ixz="0" iyy="1e-5" iyz="0" izz="1e-5"/>
+    </inertial>
+    <visual>
+      <geometry>
+        <box size="0.02 0.02 0.02"/>
+      </geometry>
+    </visual>
+  </link>
+  <joint name="scene_camera_joint" type="fixed">
+    <parent link="panda_link0"/>
+    <child link="scene_camera_link"/>
+    <origin xyz="1 0 1" rpy="3.1415 2.355 0"/>
+  </joint>
+  <gazebo reference="scene_camera_link">
+  <sensor type="camera" name="scene_camera">
+    <update_rate>30.0</update_rate>
+    <camera>
+      <horizontal_fov>1.3962634</horizontal_fov>
+      <image>
+        <width>640</width>
+        <height>480</height>
+        <format>R8G8B8</format>
+      </image>
+      <clip>
+        <near>0.1</near>
+        <far>100</far>
+      </clip>
+    </camera>
+    <plugin name="camera_controller" filename="libgazebo_ros_camera.so">
+      <alwaysOn>true</alwaysOn>
+      <updateRate>30.0</updateRate>
+      <cameraName>scene_camera</cameraName>
+      <imageTopicName>image_raw</imageTopicName>
+      <cameraInfoTopicName>camera_info</cameraInfoTopicName>
+      <frameName>scene_camera_link</frameName>
+    </plugin>
+  </sensor>
+  </gazebo>
 </robot>

Commit message: Adjust camera per libero example

File: franka_ros/franka_description/robots/panda/panda.urdf.xacro (robot description, xacro)
@@ -21,5 +21,5 @@
     <parent link="panda_hand"/>
     <child link="ee_camera_link"/>
-    <origin xyz="0.04 0 0.05" rpy="0 -2.1 0"/>
+    <origin xyz="0.03 0 0.03" rpy="3.14159 -1.45 0"/>
   </joint>
   <gazebo reference="ee_camera_link">
@@ -63,5 +63,5 @@
     <parent link="panda_link0"/>
     <child link="scene_camera_link"/>
-    <origin xyz="1 0 1" rpy="3.1415 2.355 0"/>
+    <origin xyz="1 0 0.9" rpy="3.1415 2.355 0"/>
   </joint>
   <gazebo reference="scene_camera_link">
@@ -76,5 +76,5 @@
       </image>
       <clip>
-        <near>0.1</near>
+        <near>0.05</near>
         <far>100</far>
       </clip>
