Commit message: Comment out panda hand and gazebo cameras

File: franka_ros/franka_description/robots/common/franka_robot.xacro (robot description, xacro)
@@ -14,5 +14,5 @@
     <xacro:include filename="$(find franka_description)/robots/common/franka_arm.xacro" />
     <xacro:franka_arm arm_id="${arm_id}" safety_distance="0.03" gazebo="$(arg gazebo)" joint_limits="${joint_limits}"/>
-    <xacro:if value="$(arg hand)">
+    <!-- <xacro:if value="$(arg hand)">
       <xacro:include filename="$(find franka_description)/robots/common/franka_hand.xacro"/>
       <xacro:franka_hand
@@ -25,5 +25,5 @@
           gazebo="$(arg gazebo)"
        />
-    </xacro:if>
+    </xacro:if> -->
     <!-- Define additional Gazebo tags -->
     <xacro:if value="$(arg gazebo)">
@@ -63,11 +63,11 @@
          tip="${arm_id}_joint8"
        />
-      <xacro:if value="$(arg hand)">
+      <!-- <xacro:if value="$(arg hand)">
         <xacro:gazebo-joint joint="${arm_id}_finger_joint1" transmission="hardware_interface/EffortJointInterface" />
         <xacro:gazebo-joint joint="${arm_id}_finger_joint2" transmission="hardware_interface/EffortJointInterface" />
-        <!-- Friction specific material for Rubber/Rubber contact -->
+        Friction specific material for Rubber/Rubber contact
         <xacro:gazebo-friction link="${arm_id}_leftfinger" mu="1.13" />
         <xacro:gazebo-friction link="${arm_id}_rightfinger" mu="1.13" />
-      </xacro:if>
+      </xacro:if> -->
       <gazebo>
         <plugin name="gazebo_ros_control" filename="libgazebo_ros_control.so">

File: franka_ros/franka_description/robots/panda/panda.urdf.xacro (robot description, xacro)
@@ -6,5 +6,5 @@
                       joint_limits="${xacro.load_yaml('$(find franka_description)/robots/panda/joint_limits.yaml')}">
   </xacro:franka_robot>
-  <link name="ee_camera_link">
+  <!-- <link name="ee_camera_link">
     <inertial>
       <mass value="0.1"/>
@@ -89,4 +89,4 @@
     </plugin>
   </sensor>
-  </gazebo>
+  </gazebo> -->
 </robot>
